Commit message: create bugs & worlds

File: simulation_ws/src/m2wr_description/urdf/m2wr.xacro (robot description, xacro)
@@ -1,14 +1,14 @@
 <?xml version="1.0" ?>
 <robot name="m2wr" xmlns:xacro="http://www.ros.org/wiki/xacro">
-  <xacro:include filename="$(find m2wr_description)/urdf/materials.xacro" />
-  <xacro:include filename="$(find m2wr_description)/urdf/m2wr.gazebo" />
-  <xacro:include filename="$(find m2wr_description)/urdf/macros.xacro" />
-  <link name="dummy"/>
-  <joint name="dummy_joint" type="fixed">
-    <parent link="dummy"/>
-    <child link="link_chassis"/>
-  </joint>
-  <link name="link_chassis">
-    <!-- pose and inertial -->
+  <xacro:include filename="$(find m2wr_description)/urdf/materials.xacro"/>
+  <xacro:include filename="$(find m2wr_description)/urdf/m2wr.gazebo"/>
+  <xacro:include filename="$(find m2wr_description)/urdf/macros.xacro"/>
+  <!-- <link name="dummy"/>
+    <joint name="dummy_joint" type="fixed">
+      <parent link="dummy"/>
+      <child link="link_chassis"/>
+    </joint>
+   <!-->
+  <link name="link_chassis"> -->
     <pose>0 0 0.1 0 0 0</pose>
     <inertial>
@@ -54,13 +54,8 @@
     </visual>
   </link>
-   <link name="sensor_laser">
+  <link name="sensor_laser">
     <inertial>
       <origin xyz="0 0 0" rpy="0 0 0" />
       <mass value="1" />
-      <!-- RANDOM INERTIA BELOW -->
-      <!--
-        OLD INERTIA VALUE - BEFORE RANDOM VALUE INSERTED USING MACROS
-        <inertia ixx="0.02" ixy="0" ixz="0" iyy="0.02" iyz="0" izz="0.02"/>
-      -->
       <xacro:cylinder_inertia mass="1" r="0.05" l="0.1" />
     </inertial>
@@ -84,7 +79,7 @@
     <child link="sensor_laser"/>
   </joint>
-  <xacro:link_wheel name="link_right_wheel" />
-  <xacro:joint_wheel name="joint_right_wheel" child="link_right_wheel" origin_xyz="-0.05 0.15 0" />
-  <xacro:link_wheel name="link_left_wheel" />
-  <xacro:joint_wheel name="joint_left_wheel" child="link_left_wheel" origin_xyz="-0.05 -0.15 0" />
+  <xacro:link_wheel name="link_right_wheel"/>
+  <xacro:joint_wheel name="joint_right_wheel" child="link_right_wheel" origin_xyz="-0.05 0.15 0"/>
+  <xacro:link_wheel name="link_left_wheel"/>
+  <xacro:joint_wheel name="joint_left_wheel" child="link_left_wheel" origin_xyz="-0.05 -0.15 0"/>
 </robot>

File: simulation_ws/src/m2wr_description/urdf/macros.xacro (robot description, xacro)
@@ -1,5 +1,5 @@
 <?xml version="1.0"?>
-<robot>
-    <macro name="link_wheel" params="name">
+<robot xmlns:xacro="http://wiki.ros.org/xacro">
+    <xacro:macro name="link_wheel" params="name">
         <link name="${name}">
             <inertial>
@@ -21,6 +21,6 @@
             </visual>
         </link>
-    </macro>
-    <macro name="joint_wheel" params="name child origin_xyz">
+    </xacro:macro>
+    <xacro:macro name="joint_wheel" params="name child origin_xyz">
       <joint name="${name}" type="continuous">
         <origin rpy="0 0 0" xyz="${origin_xyz}"/>
@@ -31,12 +31,9 @@
         <joint_properties damping="1.0" friction="1.0"/>
       </joint>
-    </macro>
-    <!-- <xacro:macro name="cylinder_inertia" params="mass r l">
-      <inertia ixx="${mass*(3*r*r+l*l)/12}" ixy = "0" ixz = "0" iyy="${mass*(3*r*r+l*l)/12}" iyz = "0" izz="${mass*(r*r)/2}" />
-    </xacro:macro> -->
-    <macro name="cylinder_inertia" params="mass r l">
+    </xacro:macro>
+    <xacro:macro name="cylinder_inertia" params="mass r l">
       <inertia  ixx="${mass*(3*r*r+l*l)/12}" ixy = "0" ixz = "0"
                 iyy="${mass*(3*r*r+l*l)/12}" iyz = "0"
                 izz="${mass*(r*r)/2}" />
-    </macro>
+    </xacro:macro>
 </robot>

File: simulation_ws/src/m2wr_description/urdf/materials.xacro (robot description, xacro)
@@ -1,27 +1,27 @@
-<?xml version = "1.0"?>
-<robot>
-    <material name="black">
-        <color rgba="0.0 0.0 0.0 1.0"/>
-    </material>
-    <material name="blue">
-        <color rgba="0.203125 0.23828125 0.28515625 1.0"/>
-    </material>
-    <material name="green">
-        <color rgba="0.0 0.8 0.0 1.0"/>
-    </material>
-    <material name="grey">
-        <color rgba="0.2 0.2 0.2 1.0"/>
-    </material>
-    <material name="orange">
-        <color rgba="1.0 0.423529411765 0.0392156862745 1.0"/>
-    </material>
-    <material name="brown">
-        <color rgba="0.870588235294 0.811764705882 0.764705882353 1.0"/>
-    </material>
-    <material name="red">
-        <color rgba="0.80078125 0.12890625 0.1328125 1.0"/>
-    </material>
-    <material name="white">
-        <color rgba="1.0 1.0 1.0 1.0"/>
-    </material>
+<?xml version="1.0" ?>
+<robot xmlns:xacro="http://www.ros.org/wiki/xacro">
+  <material name="black">
+    <color rgba="0.0 0.0 0.0 1.0"/>
+  </material>
+  <material name="blue">
+    <color rgba="0.203125 0.23828125 0.28515625 1.0"/>
+  </material>
+  <material name="green">
+    <color rgba="0.0 0.8 0.0 1.0"/>
+  </material>
+  <material name="grey">
+    <color rgba="0.2 0.2 0.2 1.0"/>
+  </material>
+  <material name="orange">
+    <color rgba="1.0 0.423529411765 0.0392156862745 1.0"/>
+  </material>
+  <material name="brown">
+    <color rgba="0.870588235294 0.811764705882 0.764705882353 1.0"/>
+  </material>
+  <material name="red">
+    <color rgba="0.80078125 0.12890625 0.1328125 1.0"/>
+  </material>
+  <material name="white">
+    <color rgba="1.0 1.0 1.0 1.0"/>
+  </material>
 </robot>

Commit message: final

File: simulation_ws/src/m2wr_description/urdf/m2wr.xacro (robot description, xacro)
@@ -4,11 +4,6 @@
   <xacro:include filename="$(find m2wr_description)/urdf/m2wr.gazebo"/>
   <xacro:include filename="$(find m2wr_description)/urdf/macros.xacro"/>
-  <!-- <link name="dummy"/>
-    <joint name="dummy_joint" type="fixed">
-      <parent link="dummy"/>
-      <child link="link_chassis"/>
-    </joint>
-   <!-->
-  <link name="link_chassis"> -->
+  <link name="link_chassis">
+    <!-- pose and inertial -->
     <pose>0 0 0.1 0 0 0</pose>
     <inertial>
